File: ProgrammableGain.kicad_sch (KiCad schematic)
At the start: 10 parts, among them Q15 NMOS, Q16 NMOS, Q17 NMOS, Q5 NMOS, Q6 NMOS

Commit message: schematics done
Parts:
- added R11, R14, R5, R58, R9: 10k, Resistor_SMD:R_0603_1608Metric_Pad0.98x0.95mm_HandSolder, symbol Device:R
- R26: value R -> 1k; footprint (none) -> Resistor_SMD:R_0603_1608Metric_Pad0.98x0.95mm_HandSolder
- R27: value R -> 3k3; footprint (none) -> Resistor_SMD:R_0603_1608Metric_Pad0.98x0.95mm_HandSolder
- R28: value R -> 4k7; footprint (none) -> Resistor_SMD:R_0603_1608Metric_Pad0.98x0.95mm_HandSolder
- R42: value R -> 6k8; footprint (none) -> Resistor_SMD:R_0603_1608Metric_Pad0.98x0.95mm_HandSolder
- R43: value R -> 8k2; footprint (none) -> Resistor_SMD:R_0603_1608Metric_Pad0.98x0.95mm_HandSolder
Connections:
- net GND: now also R11.2, R14.2, R5.2, R58.2, R9.2
- net PGA_GATE0: now also R5.1
- net PGA_GATE1: now also R9.1
- net PGA_GATE2: now also R11.1
- net PGA_GATE3: now also R14.1
- net PGA_GATE4: now also R58.1
Other:
- moved on the sheet: Q15, Q16, Q17, Q5, Q6, R26, R27, R28, R42, R43
