File: fpga.kicad_sch (KiCad schematic)
At the start: 51 parts, among them U1 MACHXO2-1200HC-4TG100C, U2 TDC_7200, X1 16MHz

Commit message: before changing MUX
Connections:
- net BRIDGE_C_HI: now also U1.52 (PR10C); no longer U1.54 (PR9C)
- net BRIDGE_C_LO: now also U1.51 (PR10D); no longer U1.53 (PR9D)
- net BRIDGE_D_HI: now also U1.54 (PR9C); no longer U1.51 (PR10D), U1.52 (PR10C)
- net SPI_LOCAL_MISO: now also U1.9 (PL4A); no longer U1.17 (PL8B), U16.2 (SO/SIO1)
- net SPI_LOCAL_MOSI: now also U1.10 (PL4B); no longer U1.16 (PL8A), U16.5 (SI/SIO0)
- net SPI_LOCAL_SCK: no longer U16.6 (SCK)
- net SRAM_HOLD: now also U1.27 (PB4C/CSSPIN); no longer U1.25 (PL10D)
- net STANBY_OSC: now also U1.7 (PL3C); no longer U1.9 (PL4A)
- net TDC_CS: now also U1.13 (PL5B/PCLKC3_1); no longer U1.19 (PL8D)
- net TDC_INTB: now also U1.8 (PL3D); no longer U1.10 (PL4B)
- net TDC_START: now also U1.16 (PL8A); no longer U1.14 (PL5C)
- net TDC_STOP: now also U1.15 (PL5D); no longer U1.13 (PL5B/PCLKC3_1)
- net TDC_TRIGG: now also U1.17 (PL8B); no longer U1.15 (PL5D)
- net SPI_FASTL_SCK: now reaches U1.20 (PL9A/PCLKT3_0)
- net SPI_FASTL_SCK: now also U16.6 (SCK)
- net SPI_FAST_MOSI: now reaches U1.21 (PL9B/PCLKC3_0)
- net SPI_FAST_MOSI: now also U16.5 (SI/SIO0)
- new net BRIDGE_D_LO: U1.53 (PR9D)
- new net SPI_FAST_MISO: U1.25 (PL10D), U16.2 (SO/SIO1)

Commit message: no errors schematic, basic routing done
Parts:
- C3, C35, C38, C39, C41, C42, C44, C45, C47, C48, C50, C51, C52: value 100n -> C
- C34: value 1n -> C
- C36, C37, C40, C43, C46, C49: value 1u -> C
- C4: value 10n -> C
- R60, R62, R63, R64, R65: value 100 -> R
- R61, R66, R71: value 10k -> R
Connections:
- net BRIDGE_AB_MUX_EN: now reaches U1.29 (PB6A)
- net BRIDGE_CD_MUX_EN: now reaches U1.30 (PB6B)
- net EN_SIGNAL_A renamed BRIDGE_A_SEL
- net EN_SIGNAL_B renamed BRIDGE_B_SEL
- net EN_SIGNAL_C renamed BRIDGE_C_SEL
- net EN_SIGNAL_D renamed BRIDGE_D_SEL
- no-connect marks 2 -> 11

Commit message: DONE - before checking
Parts:
- added R83, R84, R85: 12, Resistor_SMD:R_0603_1608Metric, symbol Device:R
Connections:
- net SPI_LOCAL_MISO: now also R83.1; no longer U1.9 (PL4A)
- net SPI_LOCAL_MOSI: now also R84.1; no longer U1.10 (PL4B)
- net SPI_LOCAL_SCK: now also R85.1; no longer U1.12 (PL5A/PCLKT3_1)
- new net: R84.2, U1.10 (PL4B)
- new net: R85.2, U1.12 (PL5A/PCLKT3_1)
- new net: R83.2, U1.9 (PL4A)
Other:
- note added: "FPGA"
- note added: "Oscillator"
- note added: "Power pins and hierarchy"
- note added: "SRAM"
- note added: "TDC"
- note added: "TVS"
- moved on the sheet: C3, C34, C35, C36, C37, C38, C39, C4, C40, C41, C42, C43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
