File: H-bridges.kicad_sch (KiCad schematic)
At the start: 64 parts, among them J2 Conn_Coaxial, J3 Conn_Coaxial, J6 Conn_Coaxial, J7 Conn_Coaxial, Q1 DMN6069SE, Q10 DMN6069SE, Q2 DMN6069SE, Q3 DMN6069SE, Q4 DMN6069SE, Q7 DMN6069SE, Q8 DMN6069SE, Q9 DMN6069SE, U10 MIC4604YM, U11 MIC4604YM, U19 TMUX7219, U20 TMUX7219, U21 TMUX7219, U22 TMUX7219, U8 MIC4604YM, U9 MIC4604YM

Commit message: V2 finished
Parts:
- added C10, C118, C119, C122, C123, C2, C90, C92: C, Capacitor_SMD:C_0603_1608Metric_Pad1.08x0.95mm_HandSolder, symbol Device:C
- added C11, C120, C121, C124, C125, C9, C91, C93: C, Capacitor_SMD:C_0805_2012Metric_Pad1.18x1.45mm_HandSolder, symbol Device:C
Connections:
- net GND: now also C10.2, C11.1, C118.2, C119.2, C120.1, C121.1, C122.2, C123.2, C124.1, C125.1, C2.2, C9.1, C90.2, C91.1, C92.2, C93.1
- net P12V: now also C10.1, C11.2, C2.1, C9.2, C90.1, C91.2, C92.1, C93.2
- net PHV: now also C118.1, C119.1, C120.2, C121.2, C122.1, C123.1, C124.2, C125.2
- net SIGNAL_UNAMPLIFIED_N: now also U20.8 (S2); no longer U22.8 (S2)
- net SIGNAL_UNAMPLIFIED_P: now also U22.8 (S2); no longer U20.8 (S2)
Other:
- moved on the sheet: C67, C68, C69, C70, C72, C74, C76, C87, J6, J7, Q1, Q10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
